File: Electronics/MountControl/_autosave-MountControl.kicad_pcb (KiCad board)
At the start: 2 copper layers, 194.1 x 115.6 mm, 21 parts

Commit message: Layout almost done
Parts:
- removed the G*** at (779.5, 525.3)
- moved G*** 39.0 mm to (499.1, 356.1)
Other:
- board text removed: "Closed loop stepper drivers"
- board text removed: "https://github.com/neatstranger/Dagerro"
