File: Electronics/MountControl/MountControl.kicad_sch (KiCad schematic)
At the start: 8 parts

Commit message: Schematic Finished
Parts:
- removed FOCUS-Motor, Filter-Wheel: R-RJ45R10P-B000, New:RJ45-TH_R-RJ45R10P-B000, symbol New:R-RJ45R10P-B000
- added 12V-Current-Sense, 24V-Current-Sense1, DEC-Current-Sense, FOCUS-Current-Sense1, RA-Current-Sense: HOJLR2512-3W-1MR-1%, New:RES-SMD_L6.4-W3.2-R2512, symbol New:HOJLR2512-3W-1MR-1%
- added 12V-Input, 24V-Input, Thermistor1, Thermistor2, Thermistor3, Thermistor4, Thermistor5: WJ500V-5.08-2P-14-00A, New:CONN-TH_2P-P5.00_WJ500V-5.08-2P, symbol New:WJ500V-5.08-2P-14-00A
- added FOCUS-Motor, Filter-Wheel: DB128V-5.08-5P-GN-S, New:CONN-TH_5P-P5.08_DIBO_DB128V-5.08-5P-GN-S, symbol New:DB128V-5.08-5P-GN-S
Connections:
- net +24V: now also 24V-Input.1, FOCUS-Motor.4
- net +5V: now also Thermistor1.1, Thermistor2.1, Thermistor3.1, Thermistor4.1, Thermistor5.1
- net GND: now also 12V-Current-Sense.1, 24V-Current-Sense1.1, DEC-Current-Sense.1, FOCUS-Current-Sense1.1, Filter-Wheel.2, Filter-Wheel.4, RA-Current-Sense.1; no longer DEC-Motor.5, RA-Motor.5
- net SCL: now also Filter-Wheel.5
- net SDA: now also Filter-Wheel.1
- net fcDirPin: now also FOCUS-Motor.3
- net fcEnPin: now also FOCUS-Motor.1
- net fcStepPin: now also FOCUS-Motor.2
- net 12vCurrent: now reaches A1.A0
- net 12vCurrent: now also 12V-Current-Sense.2, 12V-Input.2
- net 24vCurrent: now reaches A1.A1
- net 24vCurrent: now also 24V-Current-Sense1.2, 24V-Input.2
- net raCurrent: now reaches A1.A2
- net raCurrent: now also RA-Motor.5, RA-Current-Sense.2
- net decCurrent: now reaches A1.A3
- net decCurrent: now also DEC-Motor.5, DEC-Current-Sense.2
- net fcCurrent: now reaches A1.A4
- net fcCurrent: now also FOCUS-Current-Sense1.2, FOCUS-Motor.5
- net at A1.A5: now also Thermistor1.2
- net at A1.A6: now also Thermistor2.2
- net at A1.A7: now also Thermistor3.2
- net at A1.A8: now also Thermistor4.2
- net at A1.A9: now also Thermistor5.2
- net FilterTx: now reaches A1.D14 (D14/TX3)
- net FilterRx: now reaches A1.D15 (D15/RX3)
- new net +12V: 12V-Input.1, Filter-Wheel.3

Commit message: Finished with routing.
Parts:
- DS3131-RTC1: renamed from DS3131-RTC; footprint (none) -> Connector_PinHeader_2.54mm:PinHeader_1x06_P2.54mm_Horizontal
- renumbered 12V-Current-Sense to 12V-Current-Sense1, 12V-Input to 12V-Input1, 24V-Input to 24V-Input1, DEC-Current-Sense to DEC-Current-Sense1, DEC-Hall-Effect to DEC-Hall-Effect1, DEC-Motor to DEC-Motor1, FOCUS-Motor to FOCUS-Motor1, Filter-Wheel to Filter-Wheel1, RA-Current-Sense to RA-Current-Sense1, RA-Hall-Effect to RA-Hall-Effect1, RA-Motor to RA-Motor1
Connections:
- net +12V: now also A1.VIN
- net +5V: now also A1.5V1 (5V), A1.5V3 (5V), A1.5V4 (5V)
- net GND: now also A1.GND1 (GND), A1.GND2 (GND), A1.GND3 (GND), A1.GND5 (GND), A1.GND6 (GND)
