File: Electronics/MountControl/MountControl.kicad_pcb (KiCad board)
At the start: 2 copper layers, 194.1 x 115.6 mm, 21 parts

Commit message: Finished with routing.
Parts:
- removed the G*** at (779.5, 525.3)
- added REF**: MountingHole_3.2mm_M3, MountingHole:MountingHole_3.2mm_M3, F.Cu at (569.0, 411.5)
- added REF**: MountingHole_3.2mm_M3, MountingHole:MountingHole_3.2mm_M3, F.Cu at (386.1, 327.7)
- added REF**: MountingHole_3.2mm_M3, MountingHole:MountingHole_3.2mm_M3, F.Cu at (386.1, 431.8)
- added REF**: MountingHole_3.2mm_M3, MountingHole:MountingHole_3.2mm_M3, F.Cu at (569.0, 327.7)
- moved G*** 39.8 mm to (499.3, 357.7)
Connections:
- A1 pad 5V1: unconnected-(A1-5V-Pad5V1) -> +5V
- A1 pad 5V3: unconnected-(A1-5V-Pad5V3) -> +5V
- A1 pad 5V4: unconnected-(A1-5V-Pad5V4) -> +5V
- A1 pad GND1: unconnected-(A1-GND-PadGND1) -> GND
- A1 pad GND2: unconnected-(A1-GND-PadGND2) -> GND
- A1 pad GND3: unconnected-(A1-GND-PadGND3) -> GND
- A1 pad GND5: unconnected-(A1-GND-PadGND5) -> GND
- A1 pad GND6: unconnected-(A1-GND-PadGND6) -> GND
- A1 pad VIN: unconnected-(A1-PadVIN) -> +12V
Routing:
- net +5V: track 0.00 -> 342.9 mm
- net +24V: track 0.00 -> 288.2 mm, vias 0 -> 2
- net /decHallInterrupt: track 0.00 -> 197.9 mm, vias 0 -> 1
- net +12V: track 0.00 -> 194.0 mm
- net /raHallInterrupt: track 0.00 -> 145.7 mm, vias 0 -> 1
- net /fcDirPin: track 0.00 -> 133.4 mm
- net /fcStepPin: track 0.00 -> 124.9 mm
- net /fcEnPin: track 0.00 -> 122.5 mm
- net /SCL: track 0.00 -> 117.9 mm, vias 0 -> 2
- net /24vCurrent: track 0.00 -> 111.0 mm
- net Net-(A1-PadA5): track 0.00 -> 97.1 mm
- net /SDA: track 0.00 -> 95.8 mm, vias 0 -> 2
- net Net-(A1-PadA9): track 0.00 -> 94.4 mm
- net Net-(A1-PadA6): track 0.00 -> 92.9 mm
- net /12vCurrent: track 0.00 -> 92.6 mm
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- added copper zone on B.Cu, net GND
- added copper zone on F.Cu, net GND
- added copper zone on In1.Cu, net GND
- added copper zone on In2.Cu, net GND
Other:
- copper layers 2 -> 4
- board text removed: "Closed loop stepper drivers"
- board text removed: "https://github.com/neatstranger/Dagerro"

Commit message: Added production files
Parts:
- added DS3131-RTC1: Conn_01x06_Socket, Connector_PinHeader_2.54mm:PinHeader_1x06_P2.54mm_Horizontal, F.Cu at (493.5, 377.2)
Routing:
- net /timingInterrupt: track 0.00 -> 65.8 mm, vias 0 -> 1
- net /SCL: track 117.9 -> 160.5 mm
- net /SDA: track 95.8 -> 133.4 mm
- net +5V: track 342.9 -> 353.2 mm
