File: Electronics/Driver/Driver.kicad_pcb (KiCad board)
At the start: 2 copper layers, 0 parts

Commit message: Added driver PCB
Parts:
- added C1: 100u, Capacitor_SMD:C_1206_3216Metric_Pad1.33x1.80mm_HandSolder, F.Cu at (138.0, 76.7)
- added C2: 0.01u, Capacitor_SMD:C_1206_3216Metric_Pad1.33x1.80mm_HandSolder, F.Cu at (138.0, 80.6)
- added C3: 0.47u, Capacitor_SMD:C_1206_3216Metric_Pad1.33x1.80mm_HandSolder, F.Cu at (152.3, 84.1)
- added DC1: DC-005-20A_C136744, COMPONENTS:DC-IN-TH_DC-005-20A, F.Cu at (125.5, 81.2)
- added DC2: DC-005-20A_C136744, COMPONENTS:DC-IN-TH_DC-005-20A, F.Cu at (174.5, 76.6)
- added H1: MountingHole_Pad, MountingHole:MountingHole_3.2mm_M3_DIN965_Pad_TopBottom, F.Cu at (121.9, 55.9)
- added H2: MountingHole_Pad, MountingHole:MountingHole_3.2mm_M3_DIN965_Pad_TopBottom, F.Cu at (121.9, 91.4)
- added H3: MountingHole_Pad, MountingHole:MountingHole_3.2mm_M3_DIN965_Pad_TopBottom, F.Cu at (177.8, 91.4)
- added H4: MountingHole_Pad, MountingHole:MountingHole_3.2mm_M3_DIN965_Pad_TopBottom, F.Cu at (177.8, 55.9)
- added R1: 0, Resistor_SMD:R_1206_3216Metric_Pad1.30x1.75mm_HandSolder, F.Cu at (156.4, 70.1)
- added R2: 0, Resistor_SMD:R_1206_3216Metric_Pad1.30x1.75mm_HandSolder, F.Cu at (156.4, 72.6)
- added R3: 0, Resistor_SMD:R_1206_3216Metric_Pad1.30x1.75mm_HandSolder, F.Cu at (147.5, 68.6)
- added R4: 0, Resistor_SMD:R_1206_3216Metric_Pad1.30x1.75mm_HandSolder, F.Cu at (150.0, 68.5)
- added R5: 0, Resistor_SMD:R_1206_3216Metric_Pad1.30x1.75mm_HandSolder, F.Cu at (156.4, 76.7)
- added R6: 0, Resistor_SMD:R_1206_3216Metric_Pad1.30x1.75mm_HandSolder, F.Cu at (156.4, 79.7)
- added U1: DRV8428RTER, COMPONENTS:WQFN-16_L3.0-W3.0-P0.50-BL-EP1.7, F.Cu at (148.1, 77.9)
- added U2: DB125-2.54-4P-GN, COMPONENTS:CONN-TH_DB125-2.54-4P-GN, F.Cu at (140.5, 96.8)
- added U3: DB125-2.54-4P-GN, COMPONENTS:CONN-TH_DB125-2.54-4P-GN, F.Cu at (181.8, 67.9)
Routing:
- net +3.3V: track 0.00 -> 70.8 mm, vias 0 -> 2
- net Net-(U1-STEP): track 0.00 -> 50.3 mm, vias 0 -> 1
- net Net-(U1-DIR): track 0.00 -> 48.0 mm, vias 0 -> 1
- net Net-(U1-EN/nFAULT): track 0.00 -> 45.3 mm, vias 0 -> 1
- net Net-(U1-nSLEEP): track 0.00 -> 44.5 mm, vias 0 -> 1
- net +24V: track 0.00 -> 22.4 mm
- net GND: track 0.00 -> 22.1 mm, vias 0 -> 81
- net Net-(U1-AOUT1): track 0.00 -> 21.8 mm
- net Net-(U1-AOUT2): track 0.00 -> 21.0 mm
- net Net-(U1-BOUT2): track 0.00 -> 20.1 mm
- net Net-(U1-BOUT1): track 0.00 -> 19.3 mm
- net Net-(U1-M0): track 0.00 -> 10.3 mm
- net Net-(U1-M1): track 0.00 -> 9.02 mm
- net Net-(U1-VREF): track 0.00 -> 8.57 mm
- added copper zone on B.Cu, net GND
- added copper zone on F.Cu, net GND
Other:
- board outline added: 70 x 50 mm
- board text added: "24v"
- board text added: "3.3"
- board text added: "3.3v"
- board text added: "DRV8428"
- board text added: "GND"
- board text added: "M0"
- board text added: "M1"
- board text added: "Stepper Motor Driver"
- board text added: "VREF C/C 0->3.3V"
- board text added: "dir"
- board text added: "nFault"
- board text added: "nSLEEP"
- board text added: "step"
